Commit message: Re-export arm brc_arm_description from solidworks

File: brc_arm_description/urdf/brc_arm_description.urdf (robot description, URDF)
Before this commit: robot brc_arm_description, 12 links, 11 joints
Links:
- removed link EEbase
- removed link LFinger
- removed link LLink1
- removed link RFinger
- removed link RLink1
- removed link carriage
- removed link midarm1
- removed link midarm2
- removed link world
- removed link wrist1
- removed link wrist2
- added link EEbase_link, mass 0.0926044760959502; collision mesh filename=package://brc_arm_description/meshes/EEbase_link.STL; visual mesh filename=package://brc_arm_description/meshes/EEbase_link.STL
- added link Lfinger_link, mass 0.052749; collision mesh filename=package://brc_arm_description/meshes/Lfinger_link.STL; visual mesh filename=package://brc_arm_description/meshes/Lfinger_link.STL
- added link Llink_link, mass 0.00668722339297277; collision mesh filename=package://brc_arm_description/meshes/Llink_link.STL; visual mesh filename=package://brc_arm_description/meshes/Llink_link.STL
- added link Rfinger_link, mass 0.052748844949343; collision mesh filename=package://brc_arm_description/meshes/Rfinger_link.STL; visual mesh filename=package://brc_arm_description/meshes/Rfinger_link.STL
- added link Rlink_link, mass 0.00668722339297277; collision mesh filename=package://brc_arm_description/meshes/Rlink_link.STL; visual mesh filename=package://brc_arm_description/meshes/Rlink_link.STL
- added link carriage_link, mass 0.44772; collision mesh filename=package://brc_arm_description/meshes/carriage_link.STL; visual mesh filename=package://brc_arm_description/meshes/carriage_link.STL
- added link midarm1_link, mass 0.8362; collision mesh filename=package://brc_arm_description/meshes/midarm1_link.STL; visual mesh filename=package://brc_arm_description/meshes/midarm1_link.STL
- added link midarm2_link, mass 0.0646775902886998; collision mesh filename=package://brc_arm_description/meshes/midarm2_link.STL; visual mesh filename=package://brc_arm_description/meshes/midarm2_link.STL
- added link wrist1_link, mass 0.419666572951629; collision mesh filename=package://brc_arm_description/meshes/wrist1_link.STL; visual mesh filename=package://brc_arm_description/meshes/wrist1_link.STL
- added link wrist2_link, mass 0.129512939632169; collision mesh filename=package://brc_arm_description/meshes/wrist2_link.STL; visual mesh filename=package://brc_arm_description/meshes/wrist2_link.STL
- link base_link: mass 127.989800714743 -> 127.99
Joints:
- removed joint EEbaseJ
- removed joint LFingerJ
- removed joint LLink1J
- removed joint RFingerJ
- removed joint RLink1J
- removed joint carriageJ
- removed joint fixed
- removed joint midarm1J
- removed joint midarm2J
- removed joint wrist1J
- removed joint wrist2J
- added joint EEbase_joint: type continuous, parent wrist2_link, child EEbase_link, origin xyz=0.10009 0 0 rpy=3.1416 -1.5708 0, axis 0 0 1
- added joint Lfinger_joint: type continuous, parent Llink_link, child Lfinger_link, origin xyz=-0.08 0 0 rpy=-1.5708 0 0, axis 0 0 1, mimic joint=Llink_joint multiplier=1 offset=0
- added joint Llink_joint: type continuous, parent EEbase_link, child Llink_link, origin xyz=-0.024 -0.011 -0.014095 rpy=0 0 0, axis 0 1 0, mimic joint=Rlink_joint multiplier=1 offset=0
- added joint Rfinger_joint: type continuous, parent Rlink_link, child Rfinger_link, origin xyz=0.08 0 0 rpy=-1.5708 0 -3.1416, axis 0 0 1, mimic joint=Rlink_joint multiplier=1 offset=0
- added joint Rlink_joint: type revolute, parent EEbase_link, child Rlink_link, origin xyz=0.024 -0.011 -0.014095 rpy=0 0 0, axis 0 1 0, limit lower=0 upper=1.67 effort=0 velocity=0
- added joint carriage_joint: type prismatic, parent base_link, child carriage_link, origin xyz=0 0 0.065 rpy=1.5708 0 0, axis 0 1 0, limit lower=0 upper=0.885 effort=0 velocity=0
- added joint midarm1_joint: type revolute, parent carriage_link, child midarm1_link, origin xyz=0 0 0.1 rpy=0 0.5236 0, axis 0 1 0, limit lower=0 upper=2.7423 effort=0 velocity=0
- added joint midarm2_joint: type revolute, parent midarm1_link, child midarm2_link, origin xyz=-0.35 0 0 rpy=0 -0.43633 0, axis 0 1 0, limit lower=0 upper=4.1888 effort=0 velocity=0
- added joint wrist1_joint: type revolute, parent midarm2_link, child wrist1_link, origin xyz=0.08 0.025 0 rpy=0 0 0, axis 0 0 1, limit lower=0 upper=1.57 effort=0 velocity=0
- added joint wrist2_joint: type revolute, parent wrist1_link, child wrist2_link, origin xyz=0.225 0 0 rpy=-3.1416 -1.2217 3.1416, axis 0 1 0, limit lower=0 upper=4.165 effort=0 velocity=0

Commit message: URDF viewier

File: brc_arm_description/urdf/brc_arm_description.urdf (robot description, URDF)
Before this commit: robot brc_arm_description, 11 links, 10 joints
Joints:
- joint midarm2_joint: limit lower=0 upper=4.1888 effort=0 velocity=0 -> lower=-4.1888 upper=0 effort=0 velocity=0

Commit message: Fix arm joints

File: brc_arm_description/urdf/brc_arm_description.urdf (robot description, URDF)
Before this commit: robot brc_arm_description, 11 links, 10 joints
Joints:
- joint EEbase_joint: origin xyz=0.10009 0 0 rpy=3.1416 -1.5708 0 -> xyz=0.10009 0 0 rpy=0 -1.5708 0
- joint Rfinger_joint: origin xyz=0.08 0 0 rpy=-1.5708 0 -3.1416 -> xyz=0 0 0 rpy=-1.5708 0 -3.1416
- joint Rlink_joint: limit lower=0 upper=1.67 effort=0 velocity=0 -> lower=-1.67 upper=0 effort=0 velocity=0
- joint midarm2_joint: limit lower=-4.1888 upper=0 effort=0 velocity=0 -> lower=-4.7124 upper=0 effort=0 velocity=0
- joint wrist1_joint: limit lower=0 upper=1.57 effort=0 velocity=0 -> lower=-1.57 upper=0 effort=0 velocity=0

Commit message: Fix URDF

File: brc_arm_description/urdf/brc_arm_description.urdf (robot description, URDF)
Before this commit: robot brc_arm_description, 11 links, 10 joints
Links:
- link Lfinger_link: mass 0.052749 -> 0.052748844949343
- link Llink_link: mass 0.00668722339297277 -> 0.00668722339297278
- link Rlink_link: mass 0.00668722339297277 -> 0.00668722339297278
Joints:
- joint Lfinger_joint: mimic joint=Llink_joint multiplier=1 offset=0 -> joint=Llink_joint multiplier=-1 offset=0; origin xyz=-0.08 0 0 rpy=-1.5708 0 0 -> xyz=-0.08 0 0 rpy=-1.5707963267949 0 0
- joint Llink_joint: mimic joint=Rlink_joint multiplier=1 offset=0 -> joint=Rlink_joint multiplier=-1 offset=0; origin xyz=-0.024 -0.011 -0.014095 rpy=0 0 0 -> xyz=-0.0239999999999998 -0.0110000000000022 -0.0140949701532812 rpy=0 0 0
- joint Rfinger_joint: origin xyz=0 0 0 rpy=-1.5708 0 -3.1416 -> xyz=0.0799999999999999 0 0 rpy=-1.5707963267949 0 -3.14159265358978
- joint Rlink_joint: limit lower=-1.67 upper=0 effort=0 velocity=0 -> lower=0 upper=1.30 effort=0 velocity=0; origin xyz=0.024 -0.011 -0.014095 rpy=0 0 0 -> xyz=0.0240000000000002 -0.0110000000000023 -0.0140949701532811 rpy=0 0 0

Commit message: servo fixes

File: brc_arm_description/urdf/brc_arm_description.urdf (robot description, URDF)
Before this commit: robot brc_arm_description, 11 links, 10 joints
Joints:
- joint wrist1_joint: limit lower=-1.57 upper=0 effort=0 velocity=0 -> lower=-1.57 upper=0.523 effort=0 velocity=0

Commit message: updated midarm2 start pos

File: brc_arm_description/urdf/brc_arm_description.urdf (robot description, URDF)
Before this commit: robot brc_arm_description, 11 links, 10 joints
Joints:
- joint midarm2_joint: origin xyz=-0.35 0 0 rpy=0 -0.43633 0 -> xyz=-0.35 0 0 rpy=0 -0.7854 0

Commit message: Update midarm 2 staring position

File: brc_arm_description/urdf/brc_arm_description.urdf (robot description, URDF)
Before this commit: robot brc_arm_description, 11 links, 10 joints
Joints:
- joint midarm1_joint: origin xyz=0 0 0.1 rpy=0 0.5236 0 -> xyz=0 0 0.1 rpy=0 0.2793 0
- joint midarm2_joint: origin xyz=-0.35 0 0 rpy=0 -0.7854 0 -> xyz=-0.35 0 0 rpy=0 -1.000 0

Commit message: fixed EE start pos

File: brc_arm_description/urdf/brc_arm_description.urdf (robot description, URDF)
Before this commit: robot brc_arm_description, 11 links, 10 joints
Joints:
- joint wrist2_joint: limit lower=0 upper=4.165 effort=0 velocity=0 -> lower=-1.9024 upper=2.2626 effort=0 velocity=0; origin xyz=0.225 0 0 rpy=-3.1416 -1.2217 3.1416 -> xyz=0.225 0 0 rpy=-3.1416 -3.1241 3.1416

Commit message: flipped ee 180deg

File: brc_arm_description/urdf/brc_arm_description.urdf (robot description, URDF)
Before this commit: robot brc_arm_description, 11 links, 10 joints
Joints:
- joint wrist2_joint: origin xyz=0.225 0 0 rpy=-3.1416 -3.1241 3.1416 -> xyz=0.225 0 0 rpy=0 -3.1241 3.1416
